Commit message: orientation fixed

File: src/aw_descriptions/j_actuators/awjoint1750/urdf/awjoint1750.urdf (robot description, URDF)
Before this commit: robot awjoint1750, 2 links, 1 joints
Joints:
- joint J17: origin xyz=0.08 0 -0.076 rpy=0 1.5708 0 -> xyz=0.08 0 +0.076 rpy=0 1.5708 0

File: src/aw_descriptions/j_actuators/awjoint2080/urdf/awjoint2080.urdf (robot description, URDF)
Before this commit: robot awjoint2080, 2 links, 1 joints
Joints:
- joint J20: origin xyz=0.069 0 -0.069 rpy=0 1.5708 0 -> xyz=0.069 0 +0.069 rpy=0 1.5708 0

File: src/aw_descriptions/j_actuators/awjoint2580/urdf/awjoint2580.urdf (robot description, URDF)
Before this commit: robot awjoint2580, 2 links, 1 joints
Joints:
- joint J25: origin xyz=0.0925 0 -0.0875 rpy=0 1.5708 0 -> xyz=0.0925 0 +0.0875 rpy=0 1.5708 0

File: src/aw_descriptions/j_actuators/awjoint32100/urdf/awjoint32100.urdf (robot description, URDF)
Before this commit: robot awjoint32100, 2 links, 1 joints
Joints:
- joint J32: origin xyz=0.1085 0 -0.1005 rpy=0 1.5708 0 -> xyz=0.1085 0 +0.1005 rpy=0 1.5708 0

File: src/aw_descriptions/j_actuators/awjoint40100/urdf/awjoint40100.urdf (robot description, URDF)
Before this commit: robot awjoint40100, 2 links, 1 joints
Joints:
- joint J40: origin xyz=0.1179 0 -0.1045 rpy=0 1.5708 0 -> xyz=0.1179 0 +0.1045 rpy=0 1.5708 0
